Commit message: Phase 6 complete: gripper and pick and place

File: src/arm_description/urdf/arm.urdf.xacro (robot description, xacro)
@@ -3,4 +3,6 @@
   <xacro:arg name="prefix" default=""/>
   <xacro:include filename="$(find arm_description)/urdf/arm_macro.xacro"/>
+  <xacro:include filename="$(find arm_description)/urdf/gripper.xacro"/>
   <xacro:arm prefix="$(arg prefix)"/>
+  <xacro:parallel_gripper prefix="$(arg prefix)" parent="$(arg prefix)tool0"/>
 </robot>

File: src/arm_description/urdf/arm_gazebo.xacro (robot description, xacro)
@@ -20,4 +20,10 @@
       <xacro:jnt n="5"/>
       <xacro:jnt n="6"/>
+      <joint name="${prefix}finger_joint">
+        <command_interface name="position"/>
+        <state_interface name="position"/>
+        <state_interface name="velocity"/>
+        <state_interface name="effort"/>
+      </joint>
     </ros2_control>
     <gazebo>

File: src/arm_description/urdf/arm_sim.urdf.xacro (robot description, xacro)
@@ -6,4 +6,5 @@
   <xacro:include filename="$(find arm_description)/urdf/arm_gazebo.xacro"/>
   <xacro:include filename="$(find arm_description)/urdf/camera.xacro"/>
+  <xacro:include filename="$(find arm_description)/urdf/gripper.xacro"/>
   <link name="world"/>
   <joint name="world_joint" type="fixed">
@@ -16,3 +17,4 @@
                     controller_config="$(arg controller_config)"/>
   <xacro:wrist_camera prefix="$(arg prefix)" parent="$(arg prefix)tool0"/>
+  <xacro:parallel_gripper prefix="$(arg prefix)" parent="$(arg prefix)tool0"/>
 </robot>
